Commit message: Add gravity compensation control mode for OpenMANIPULATOR-X, including new launch files, configuration for hardware controller manager, and a shutdown torque disable script.

File: open_manipulator_description/gazebo/open_manipulator_x.gazebo.xacro (robot description, xacro)
@@ -1,6 +1,6 @@
 <?xml version="1.0"?>
 <robot xmlns:xacro="http://ros.org/wiki/xacro">
-  <xacro:macro name="open_manipulator_x_gazebo" params="prefix">
-  <xacro:macro name="SimpleTransmission" params="trans joint actuator">
+  <xacro:macro name="open_manipulator_x_gazebo" params="prefix use_effort_transmission:=false">
+  <xacro:macro name="PositionTransmission" params="trans joint actuator">
     <transmission name="${trans}">
       <type>transmission_interface/SimpleTransmission</type>
@@ -11,4 +11,16 @@
         <mechanicalReduction>1</mechanicalReduction>
         <hardwareInterface>PositionJointInterface</hardwareInterface>
+      </actuator>
+    </transmission>
+  </xacro:macro>
+  <xacro:macro name="EffortTransmission" params="trans joint actuator">
+    <transmission name="${trans}">
+      <type>transmission_interface/SimpleTransmission</type>
+      <joint name="${joint}">
+        <hardwareInterface>EffortJointInterface</hardwareInterface>
+      </joint>
+      <actuator name="${actuator}">
+        <mechanicalReduction>1</mechanicalReduction>
+        <hardwareInterface>EffortJointInterface</hardwareInterface>
       </actuator>
     </transmission>
@@ -33,10 +45,18 @@
   <gazebo reference="${prefix}end_effector_link">
   </gazebo>
-  <xacro:SimpleTransmission trans="${prefix}trans1" joint="${prefix}joint1" actuator="${prefix}actuator1" />
-  <xacro:SimpleTransmission trans="${prefix}trans2" joint="${prefix}joint2" actuator="${prefix}actuator2" />
-  <xacro:SimpleTransmission trans="${prefix}trans3" joint="${prefix}joint3" actuator="${prefix}actuator3" />
-  <xacro:SimpleTransmission trans="${prefix}trans4" joint="${prefix}joint4" actuator="${prefix}actuator4" />
-  <xacro:SimpleTransmission trans="${prefix}trans5" joint="${prefix}gripper_left_joint" actuator="${prefix}actuator5" />
-  <xacro:SimpleTransmission trans="${prefix}trans6" joint="${prefix}gripper_right_joint" actuator="${prefix}actuator6" />
+  <xacro:if value="${use_effort_transmission}">
+    <xacro:EffortTransmission trans="${prefix}trans1" joint="${prefix}joint1" actuator="${prefix}actuator1" />
+    <xacro:EffortTransmission trans="${prefix}trans2" joint="${prefix}joint2" actuator="${prefix}actuator2" />
+    <xacro:EffortTransmission trans="${prefix}trans3" joint="${prefix}joint3" actuator="${prefix}actuator3" />
+    <xacro:EffortTransmission trans="${prefix}trans4" joint="${prefix}joint4" actuator="${prefix}actuator4" />
+  </xacro:if>
+  <xacro:unless value="${use_effort_transmission}">
+    <xacro:PositionTransmission trans="${prefix}trans1" joint="${prefix}joint1" actuator="${prefix}actuator1" />
+    <xacro:PositionTransmission trans="${prefix}trans2" joint="${prefix}joint2" actuator="${prefix}actuator2" />
+    <xacro:PositionTransmission trans="${prefix}trans3" joint="${prefix}joint3" actuator="${prefix}actuator3" />
+    <xacro:PositionTransmission trans="${prefix}trans4" joint="${prefix}joint4" actuator="${prefix}actuator4" />
+  </xacro:unless>
+  <xacro:PositionTransmission trans="${prefix}trans5" joint="${prefix}gripper_left_joint" actuator="${prefix}actuator5" />
+  <xacro:PositionTransmission trans="${prefix}trans6" joint="${prefix}gripper_right_joint" actuator="${prefix}actuator6" />
   </xacro:macro>
 </robot>

File: open_manipulator_description/urdf/open_manipulator_x/open_manipulator_x.urdf.xacro (robot description, xacro)
@@ -7,4 +7,6 @@
   <xacro:arg name="port_name" default="/dev/ttyUSB0" />
   <xacro:arg name="ros2_control_type" default="open_manipulator_x_position" />
+  <xacro:arg name="config_type" default="open_manipulator_x" />
+  <xacro:arg name="use_effort_transmission" default="false" />
   <xacro:include filename="$(find open_manipulator_description)/gazebo/open_manipulator_x.gazebo.xacro" />
   <xacro:include filename="$(find open_manipulator_description)/urdf/open_manipulator_x/open_manipulator_x_arm.urdf.xacro" />
@@ -17,5 +19,7 @@
   </joint>
   <xacro:open_manipulator_x prefix="$(arg prefix)" />
-  <xacro:open_manipulator_x_gazebo prefix="$(arg prefix)" />
+  <xacro:open_manipulator_x_gazebo
+    prefix="$(arg prefix)"
+    use_effort_transmission="$(arg use_effort_transmission)" />
   <xacro:open_manipulator_x_system
     name="OpenManipulatorXSystem" prefix="$(arg prefix)" use_sim="$(arg use_sim)"
@@ -25,5 +29,5 @@
   <gazebo>
     <plugin filename="gz_ros2_control-system" name="gz_ros2_control::GazeboSimROS2ControlPlugin">
-      <parameters>$(find open_manipulator_bringup)/config/open_manipulator_x/hardware_controller_manager.yaml</parameters>
+      <parameters>$(find open_manipulator_bringup)/config/$(arg config_type)/hardware_controller_manager.yaml</parameters>
     </plugin>
   </gazebo>
